Commit message: Update robot.xacro

File: urdf/robot.xacro (robot description, xacro)
@@ -1,146 +1,75 @@
 <?xml version="1.0"?>
 <robot xmlns:xacro="http://www.ros.org/wiki/xacro" name="navvis">
- <link name="base">
-  <visual>
-   <origin xyz="0.0 0.0 0.96" rpy="0.0 0.0 0.0" />
-   <geometry>
-    <box size="0.45 0.78 1.92" />
-   </geometry>
-  </visual>
-  <collision>
-   <origin xyz="0.0 0.0 0.96" rpy="0.0 0.0 0.0" />
-   <geometry>
-    <box size="0.45 0.78 1.92" />
-   </geometry>
-  </collision>
- </link>
-  <joint name="base_laser_horiz" type="fixed">
-  <parent link="base" />
-  <child link="laser_horiz" />
-  <origin xyz="0.2325 0.0001 1.9201" rpy="-0.0012 0.1146 -0.0015" />
- </joint>
-  <link name="laser_horiz">
-  <visual>
-    <origin xyz="0.2325 0.0001 1.9201" rpy="-0.0012 0.1146 -0.0015" />
-    <geometry>
-     <cylinder radius="0.052" length="0.072" />
-    </geometry>
-   </visual>
-   <collision>
-    <origin xyz="0.2325 0.0001 1.9201" rpy="-0.0012 0.1146 -0.0015" />
-    <geometry>
-     <cylinder radius="0.052" length="0.072" />
-    </geometry>
-   </collision>
-  </link>
-  <joint name="base_laser_vert_top_left" type="fixed">
-  <parent link="base" />
-  <child link="laser_vert_top_left" />
-  <origin xyz="0.2997 0.1531 1.8443" rpy="1.1780 0.6198 1.9560" />
- </joint>
-  <link name="laser_vert_top_left">
-  <visual>
-    <origin xyz="0.2997 0.1531 1.8443" rpy="1.1780 0.6198 1.9560" />
-    <geometry>
-     <box size="0.062 0.062 0.087" />
-    </geometry>
-   </visual>
-   <collision>
-    <origin xyz="0.2997 0.1531 1.8443" rpy="1.1780 0.6198 1.9560" />
-    <geometry>
-     <box size="0.062 0.062 0.087" />
-    </geometry>
-   </collision>
-  </link>
-  <joint name="base_laser_vert_top_right" type="fixed">
-  <parent link="base" />
-  <child link="laser_vert_top_right" />
-  <origin xyz="0.2978 -0.1450 1.8451" rpy="-1.1760 0.6313 -1.9377" />
- </joint>
- <link name="laser_vert_top_right">
-  <visual>
-    <origin xyz="0.2978 -0.1450 1.8451" rpy="-1.1760 0.6313 -1.9377" />
-    <geometry>
-     <box size="0.062 0.062 0.087" />
-    </geometry>
-   </visual>
-   <collision>
-    <origin xyz="0.2978 -0.1450 1.8451" rpy="-1.1760 0.6313 -1.9377" />
-    <geometry>
-     <box size="0.062 0.062 0.087" />
-    </geometry>
-   </collision>
- </link>
- <joint name="base_laser_vert_bottom_joint" type="fixed">
-  <parent link="base" />
-  <child link="laser_vert_bottom" />
-  <origin xyz="0.3158 -0.0021 0.5100" rpy="3.1355 -1.3045 0.0025" />
- </joint>
- <link name="laser_vert_bottom">
- <visual>
-   <origin xyz="0.3158 -0.0021 0.5100" rpy="3.1355 -1.3045 0.0025" />
-   <geometry>
-    <box size="0.062 0.062 0.087" />
-   </geometry>
-  </visual>
-  <collision>
-   <origin xyz="0.3158 -0.0021 0.5100" rpy="3.1355 -1.3045 0.0025" />
-   <geometry>
-    <box size="0.062 0.062 0.087" />
-   </geometry>
-  </collision>
- </link>
- <link name ="wheel_center">
-    <visual>
-      <origin xyz="0.0 0.0 0.0" rpy="0.0 0.0 0.0" />
-      <geometry>
-        <cylinder radius="0.15" length="0.05" />
-      </geometry>
-    </visual>
-    <collision>
-      <origin xyz="0.0 0.0 0.0" rpy="0.0 0.0 0.0" />
-      <geometry>
-	<cylinder radius="0.15" length="0.05" />
-      </geometry>
-    </collision>
-  </link>
-  <joint name="base_wheel_center_joint" type="continuous">
-    <parent link="base" />
-    <child link="wheel_center" />
-    <axis xyz="0 0 1" />
-    <origin xyz="0.10 0.0 -0.05" rpy="${-pi/2} 0.0 0.0" />
-    <limit effort="100" velocity="100" />
-  </joint>
- <xacro:macro name="xacro_name" params="side reflect">
-  <link name="wheel_${side}">
-   <visual>
-    <origin xyz="-0.10 0.4 0.0" rpy="{-pi/2} 0.0 0.0" />
-    <geometry>
-     <cylinder radius="0.2" length="0.05" />
-    </geometry>
-   </visual>
-   <collision>
-    <origin xyz="-0.10 0.4 0.0" rpy="{-pi/2} 0.0 0.0" />
-    <geometry>
-     <cylinder radius="0.2" length="0.05" />
-    </geometry>
-   </collision>
-  </link>
-  <joint name="base_wheel_${side}_joint" type="continuous">
-   <parent link="base" />
-   <child link="wheel_${side}" />
-   <axis xyz = "0 0 1"/>
-   <origin xyz="-0.10 ${reflect * 0.4} 0.0" rpy="${-pi/2} 0.0 0.0" />
-   <limit effort="100" velocity="100" />
-  </joint>
- </xacro:macro>
- <xacro:include filename="$(find gazebo_plugins)/test/multi_robot_scenario/xacro/laser/hokuyo.xacro" />
-  <xacro:laser name="laser_vert_bottom" parent="base" xyz="0.3157894464801903 -0.002068548615034871 0.5099999434059285" rpy="3.1354753 -1.3045001 0.0024658" meshes="package://gazebo_plugins/test/multi_robot_scenario/meshes/laser" />
-  <xacro:laser name="laser_vert_top_right" parent="base" xyz="0.2978 -0.1450 1.8451" rpy="-1.1760 0.6313 -1.9377" meshes="package://gazebo_plugins/test/multi_robot_scenario/meshes/laser" />
-  <xacro:laser name="laser_vert_top_left" parent="base" xyz="0.2997 0.1531 1.8443" rpy="1.1780 0.6198 1.9560" meshes="package://gazebo_plugins/test/multi_robot_scenario/meshes/laser" />
-  <xacro:include filename="$(find velodyne_description)/urdf/VLP-16.urdf.xacro" />
-  <xacro:VLP-16 parent="base" name="laser_horiz" topic="laser_horiz/packets" hz="10" samples="440" gpu="false"> <origin xyz="0.2325416305773505 -0.0001380069427607134 1.920122926231907" rpy="-0.0012068 0.114646 -0.0015308" />
-  </xacro:VLP-16>
- <xacro:xacro_name side="left" reflect="1" />
- <xacro:xacro_name side="right" reflect="-1" />
+    <link name="base">
+        <visual>
+            <origin xyz="0.0 0.0 0.96" rpy="0.0 0.0 0.0" />
+            <geometry>
+                <box size="0.45 0.78 1.92" />
+            </geometry>
+        </visual>
+        <collision>
+            <origin xyz="0.0 0.0 0.96" rpy="0.0 0.0 0.0" />
+            <geometry>
+                <box size="0.45 0.78 1.92" />
+            </geometry>
+        </collision>
+    </link>
+    <!-- Include other files -->
+    <xacro:include filename="$(find gazebo_plugins)/test/multi_robot_scenario/xacro/laser/hokuyo.xacro" />
+    <xacro:include filename="$(find velodyne_description)/urdf/VLP-16.urdf.xacro" />
+    <xacro:laser name="laser_vert_bottom" parent="base" xyz="0.3157894464801903 -0.002068548615034871 0.5099999434059285" rpy="3.1354753 -1.3045001 0.0024658" meshes="package://gazebo_plugins/test/multi_robot_scenario/meshes/laser" />
+    <xacro:laser name="laser_vert_top_left" parent="base" xyz="0.2997 0.1531 1.8443" rpy="1.1780 0.6198 1.9560" meshes="package://gazebo_plugins/test/multi_robot_scenario/meshes/laser" />
+    <xacro:laser name="laser_vert_top_right" parent="base" xyz="0.2978 -0.1450 1.8451" rpy="-1.1760 0.6313 -1.9377" meshes="package://gazebo_plugins/test/multi_robot_scenario/meshes/laser" />
+    <xacro:VLP-16 parent="base" name="laser_horiz" topic="laser_horiz/packets" hz="10" samples="440" gpu="false">
+        <origin xyz="0.2325416305773505 -0.0001380069427607134 1.920122926231907" rpy="-0.0012068 0.114646 -0.0015308" />
+    </xacro:VLP-16>
+    <!-- Link and joint of wheel_center !-->
+    <link name="wheel_center">
+        <visual>
+            <origin xyz="0.0 0.0 0.0" rpy="0.0 0.0 0.0"/>
+            <geometry>
+                <cylinder radius="0.15" length="0.05"/>
+            </geometry>
+        </visual>
+        <collision>
+            <origin xyz="0.0 0.0 0.0" rpy="0.0 0.0 0.0"/>
+            <geometry>
+                <cylinder radius="0.15" length="0.05"/>
+            </geometry>
+        </collision>
+    </link>
+    <joint name="base_wheel_center_joint" type="continuous">
+        <parent link="base" />
+        <child link="wheel_center" />
+        <origin xyz="0.10 0.0 -0.05" rpy="-1.57079632679 0.0 0.0" />
+        <limit effort="1000.0" velocity="80.0"/>
+        <axis xyz="0.0 0.0 1.0"/>
+    </joint>
+    <!-- Define the macro for the wheel link and joint !-->
+    <xacro:macro name="xacro_name" params="side reflect">
+        <joint name="base_wheel_${side}_joint" type="fixed">
+            <parent link="base" />
+            <child link="wheel_${side}" />
+            <origin xyz="-0.10 ${reflect * 0.4} 0.0" rpy="-1.57079632679 0.0 0.0" />
+            <limit effort="1000.0" velocity="80.0"/>
+            <axis xyz="0.0 0.0 1.0"/>
+        </joint>
+        <link name="wheel_${side}">
+            <visual>
+                <origin xyz="0.0 0.0 0.0" rpy="0.0 0.0 0.0"/>
+                <geometry>
+                    <cylinder radius="0.2" length="0.05"/>
+                </geometry>
+            </visual>
+            <collision>
+                <origin xyz="0.0 0.0 0.0" rpy="0.0 0.0 0.0"/>
+                <geometry>
+                    <cylinder radius="0.2" length="0.05"/>
+                </geometry>
+            </collision>
+        </link>
+    </xacro:macro>
+    <!-- Call the XACRO Macro. !-->
+    <xacro:xacro_name side="left" reflect="1" />
+    <xacro:xacro_name side="right" reflect="-1" />
 </robot>
